File: kicad/megabusmaster.kicad_pcb (KiCad board)
At the start: 2 copper layers, 130.8 x 111.8 mm, 46 parts, among them J1 Conn_02x32_Odd_Even, J10 Conn_01x08_Pin, J11 Conn_01x13_Pin, J12 Conn_01x13_Pin, J13 Conn_01x06_Pin, J14 Conn_01x04_Pin, J15 Conn_01x02_Pin, J2 Conn_01x06_Pin, J3 Conn_02x04_Odd_Even, J4 Conn_02x10_Odd_Even, J5 Conn_01x09_Pin, J6 Conn_01x09_Pin, J7 Conn_01x08_Pin, J8 Conn_01x08_Pin, J9 Conn_01x08_Pin, U1 MC68000P, U2 LM1117T-3.3, U3 XC9572XL-xxVQx44, U4 GAL16V8, U5 GAL16V8, U6 GAL20V8, U7 GAL20V8

Commit message: Version 0.1 as ordered.
Other:
- board text added: "CPLD-BUFFERED CLOCK MOTHERBOARD CLOCK"
- board text added: "IPL1 IPL2"
- board text removed: "DO SILKSCREEN"
Changed lines of the file:
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@@
 			(drillshape 0)
 			(scaleselection 1)
-			(outputdirectory "preview")
+			(outputdirectory "mbm_0.1")
 		)
 	)
@@
 			(at 0 -4.15 0)
 			(layer "F.SilkS")
+			(hide yes)
 			(effects
 				(font
@@
 			(at 0 -4.15 0)
 			(layer "F.SilkS")
+			(hide yes)
 			(effects
 				(font
@@
 		)
 		(embedded_fonts no)
-		(model "${KICAD9_3DMODEL_DIR}/Package_DIP.3dshapes/DIP-64_W22.86mm.step"
+		(model "${KICAD9_3DMODEL_DIR}/Package_DIP.3dshapes/DIP-64_W22.86mm_Socket.wrl"
+			(hide yes)
 			(offset
 				(xyz 0 0 0)
@@
 			(at 0 -4.15 0)
 			(layer "F.SilkS")
+			(hide yes)
 			(effects
 				(font
@@
 			(at 0 -4.15 0)
 			(layer "F.SilkS")
+			(hide yes)
 			(effects
 				(font
@@
 	)
 	(gr_line
-		(start 29.21 160.02)
-		(end 29.21 57.15)
+		(start 56.515 148.59)
+		(end 56.515 151.13)
 		(stroke
 			(width 0.1)
 			(type default)
 		)
-		(layer "Dwgs.User")
+		(layer "F.SilkS")
 	)
 	(gr_line
-		(start 29.21 160.02)
-		(end 160.02 160.02)
+		(start 56.515 152.4)
+		(end 56.515 154.94)
 		(stroke
 			(width 0.1)
 			(type default)
 		)
-		(layer "Dwgs.User")
+		(layer "F.SilkS")
+	)
+	(gr_line
+		(start 56.515 151.13)
+		(end 56.515 151.13)
+		(stroke
+			(width 0.1)
+			(type default)
+		)
+		(layer "F.SilkS")
 	)
 	(gr_line
@@
 	)
 	(gr_line
+		(start 29.21 160.02)
+		(end 160.02 160.02)
+		(stroke
+			(width 0.1)
+			(type default)
+		)
+		(layer "Dwgs.User")
+	)
+	(gr_line
 		(start 152.4 144.78)
 		(end 152.4 26.67)
@@
 		(layer "Dwgs.User")
 	)
+	(gr_line
+		(start 29.21 160.02)
+		(end 29.21 57.15)
+		(stroke
+			(width 0.1)
+			(type default)
+		)
+		(layer "Dwgs.User")
+	)
 	(gr_rect
 		(start 25.4 53.34)
@@
 		(layer "Edge.Cuts")
 	)
-	(gr_text "PULLED TO 5V (bus)"
-		(at 37.465 75.565 90)
+	(gr_text "12V GND GND GND 5V 5V"
+		(at 155.575 135.89 90)
 		(layer "F.SilkS")
 		(effects
@@
 		)
 	)
-	(gr_text "12V GND GND GND 5V 5V"
-		(at 155.575 135.89 90)
+	(gr_text "5V\nGND"
+		(at 151.765 102.235 270)
 		(layer "F.SilkS")
 		(effects
 			(font
-				(size 1 0.762)
-				(thickness 0.1524)
+				(size 1.27 1)
+				(thickness 0.2)
+				(bold yes)
+			)
+			(justify right)
+		)
+	)
+	(gr_text "IPL1 IPL2"
+		(at 48.34 162.78 0)
+		(layer "F.SilkS")
+		(effects
+			(font
+				(size 1 1)
+				(thickness 0.2)
 				(bold yes)
 			)
@@
 		)
 	)
-	(gr_text "5V\nGND"
-		(at 151.765 102.235 270)
+	(gr_text "CPLD-BUFFERED CLOCK\n\nMOTHERBOARD CLOCK"
+		(at 56.81 154.115 0)
 		(layer "F.SilkS")
 		(effects
 			(font
-				(size 1.27 1)
+				(size 1 1)
 				(thickness 0.2)
 				(bold yes)
 			)
-			(justify right)
+			(justify left bottom)
 		)
 	)
@@
 		)
 	)
-	(gr_text "DO SILKSCREEN"
-		(at 80.01 125.095 0)
-		(layer "User.4")
+	(gr_text "PULLED TO 5V (bus)"
+		(at 37.465 75.565 90)
+		(layer "F.SilkS")
 		(effects
 			(font
-				(size 3.048 3.048)
-				(thickness 0.15)
+				(size 1 0.762)
+				(thickness 0.1524)
+				(bold yes)
 			)
 			(justify left bottom)

Commit message: Started board layout of rev2
Parts:
- removed J10, J7, J8, J9: Conn_01x08_Pin, Connector_PinHeader_2.54mm:PinHeader_1x08_P2.54mm_Vertical
- removed J11, J12: Conn_01x13_Pin, Connector_PinHeader_2.54mm:PinHeader_1x13_P2.54mm_Vertical
- removed J14: Conn_01x04_Pin, Connector_PinHeader_2.54mm:PinHeader_1x04_P2.54mm_Vertical
- removed J6: Conn_01x09_Pin, Connector_PinHeader_2.54mm:PinHeader_1x09_P2.54mm_Vertical
- removed R5, R6: 10k, Resistor_SMD:R_0805_2012Metric_Pad1.20x1.40mm_HandSolder
- removed U4, U5: GAL16V8, Package_DIP:DIP-20_W7.62mm_Socket_LongPads
- removed U6, U7: GAL20V8, Package_DIP:DIP-24_W7.62mm_Socket_LongPads
- added C13: 100n, Capacitor_SMD:C_0805_2012Metric_Pad1.18x1.45mm_HandSolder, F.Cu at (207.2, 104.3)
- added C14: 100n, Capacitor_SMD:C_0805_2012Metric_Pad1.18x1.45mm_HandSolder, F.Cu at (207.2, 107.3)
- added C15: 100n, Capacitor_SMD:C_0805_2012Metric_Pad1.18x1.45mm_HandSolder, F.Cu at (207.2, 110.3)
- added IC1: SN74CB3T3245PW, Package_SO:TSSOP-20_4.4x6.5mm_P0.65mm, F.Cu at (105.4, 148.6)
- added IC2: SN74CB3T3245PW, Package_SO:TSSOP-20_4.4x6.5mm_P0.65mm, F.Cu at (120.9, 148.7)
- added IC3: SN74CB3T3245PW, Package_SO:TSSOP-20_4.4x6.5mm_P0.65mm, F.Cu at (110.1, 186.4)
- added IC4: SN74CB3T3245PW, Package_SO:TSSOP-20_4.4x6.5mm_P0.65mm, F.Cu at (62.9, 148.6)
- added IC5: SN74CB3T3245PW, Package_SO:TSSOP-20_4.4x6.5mm_P0.65mm, F.Cu at (74.3, 148.6)
- added IC6: SN74CB3T3245PW, Package_SO:TSSOP-20_4.4x6.5mm_P0.65mm, F.Cu at (85.7, 148.6)
- added R10: 10k, Resistor_SMD:R_0805_2012Metric_Pad1.20x1.40mm_HandSolder, F.Cu at (212.0, 106.9)
- added R8: 10k, Resistor_SMD:R_0805_2012Metric_Pad1.20x1.40mm_HandSolder, F.Cu at (212.0, 101.0)
- added R9: 10k, Resistor_SMD:R_0805_2012Metric_Pad1.20x1.40mm_HandSolder, F.Cu at (212.0, 104.0)
- J4: value Conn_02x10_Odd_Even -> Conn_02x07_Counter_Clockwise; footprint Connector_PinHeader_2.54mm:PinHeader_2x10_P2.54mm_Vertical -> Package_DIP:DIP-14_W7.62mm_Socket
- J5: value Conn_01x09_Pin -> Conn_02x03_Odd_Even; footprint Connector_PinHeader_2.54mm:PinHeader_1x09_P2.54mm_Vertical -> Connector_PinHeader_2.54mm:PinHeader_2x03_P2.54mm_Vertical
- R2: value 10k -> 1k
- moved R1 178.7 mm to (212.0, 92.2), turned to 0 degrees
- moved R3 159.1 mm to (212.0, 95.1), turned to 0 degrees
- moved C6 146.0 mm to (207.2, 92.2)
- moved R4 129.3 mm to (212.0, 98.1), turned to 0 degrees
- moved C7 118.1 mm to (207.2, 95.2)
- moved C8 90.4 mm to (207.2, 98.2)
- moved C9 65.7 mm to (207.2, 101.2)
- moved J5 52.9 mm to (29.1, 116.9)
- moved J4 29.8 mm to (29.2, 94.6), turned to 0 degrees
- moved R7 22.9 mm to (144.5, 146.3)
- moved C2 9.93 mm to (98.4, 120.9), turned to -90 degrees
Connections:
- net /CLK8_I renamed /CLK8I
- J1 pad 1: /D4 -> /DM4
- J1 pad 10: /D9 -> /DM9
- J1 pad 11: /~{AS} -> /~{AS}M
- J1 pad 12: /D10 -> /DM10
- J1 pad 13: /~{UDS} -> /~{UDS}M
- J1 pad 14: /D11 -> /DM11
- J1 pad 15: /~{LDS} -> /~{LDS}M
- J1 pad 16: /D12 -> /DM12
- J1 pad 17: /R~{W} -> /R~{W}M
- J1 pad 18: /D13 -> /DM13
- J1 pad 19: /~{DTACK} -> /~{DTACK}M
- J1 pad 2: /D5 -> /DM5
- J1 pad 20: /D14 -> /DM14
- J1 pad 21: /~{BG_MB} -> /~{BG_MB}M
- J1 pad 22: /D15 -> /DM15
- J1 pad 23: /~{BGACK_MB} -> /~{BGACK_MB}M
- J1 pad 25: /~{BR_MB} -> /~{BR_MB}M
- J1 pad 26: /A23 -> /AM23
- J1 pad 28: /A22 -> /AM22
- J1 pad 29: /CLK8 -> /CLK8M
- J1 pad 3: /D3 -> /DM3
- J1 pad 30: /A21 -> /AM21
- J1 pad 33: /~{HALT_MB} -> /~{HALT_MB}M
- J1 pad 34: /A20 -> /AM20
- J1 pad 35: /~{RESET_MB} -> /~{RESET}
- J1 pad 36: /A19 -> /AM19
- J1 pad 37: /~{VMA} -> /~{VMA}M
- J1 pad 38: /A18 -> /AM18
- J1 pad 39: /E -> /EM
- J1 pad 4: /D6 -> /DM6
- J1 pad 40: /A17 -> /AM17
- J1 pad 41: /~{VPA} -> /~{VPA}M
- J1 pad 42: /A16 -> /AM16
- J1 pad 43: /~{BERR} -> /~{BERR}M
- J1 pad 44: /A15 -> /AM15
- J1 pad 46: /A14 -> /AM14
- J1 pad 48: /A13 -> /AM13
- J1 pad 5: /D2 -> /DM2
- J1 pad 50: /A12 -> /AM12
- J1 pad 51: /~{FC2} -> /~{FC2}M
- J1 pad 52: /A11 -> /AM11
- J1 pad 53: /~{FC1} -> /~{FC1}M
- J1 pad 54: /A10 -> /AM10
- J1 pad 55: /~{FC0} -> /~{FC0}M
- J1 pad 56: /A9 -> /AM9
- J1 pad 57: /A1 -> /AM1
- J1 pad 58: /A8 -> /AM8
- J1 pad 59: /A2 -> /AM2
- J1 pad 6: /D7 -> /DM7
- J1 pad 60: /A7 -> /AM7
- J1 pad 61: /A3 -> /AM3
- J1 pad 62: /A6 -> /AM6
- J1 pad 63: /A4 -> /AM4
- J1 pad 64: /A5 -> /AM5
- J1 pad 7: /D1 -> /DM1
- J1 pad 8: /D8 -> /DM8
- J1 pad 9: /D0 -> /DM0
- J4 pad 1: /~{RESET_MB} -> unconnected-(J4-Pin_1-Pad1)
- J4 pad 10: /~{BG_MB_CPLD} -> unconnected-(J4-Pin_10-Pad10)
- J4 pad 11: /~{BG_I} -> /OSC
- J4 pad 12: /~{BG_I_CPLD} -> unconnected-(J4-Pin_12-Pad12)
- J4 pad 13: /~{BGACK_I} -> unconnected-(J4-Pin_13-Pad13)
- J4 pad 14: /~{BGACK_I_CPLD} -> +5V
- J4 pad 2: /~{RESET_MB_CPLD} -> unconnected-(J4-Pin_2-Pad2)
- J4 pad 3: /~{HALT_MB} -> unconnected-(J4-Pin_3-Pad3)
- J4 pad 4: /~{HALT_MB_CPLD} -> GND
- J4 pad 5: /~{BR_MB} -> unconnected-(J4-Pin_5-Pad5)
- J4 pad 6: /~{BR_MB_CPLD} -> unconnected-(J4-Pin_6-Pad6)
- J4 pad 7: /~{BGACK_MB} -> GND
- J4 pad 8: /~{BGACK_MB_CPLD} -> /OSC
- J4 pad 9: /~{BG_MB} -> unconnected-(J4-Pin_9-Pad9)
- J5 pad 1: Net-(J5-Pin_1) -> /CONFIG0
- J5 pad 2: Net-(J5-Pin_2) -> GND
- J5 pad 3: Net-(J5-Pin_3) -> /CONFIG1
- J5 pad 4: Net-(J5-Pin_4) -> GND
- J5 pad 5: Net-(J5-Pin_5) -> /CONFIG2
- J5 pad 6: Net-(J5-Pin_6) -> GND
- JP1 pad 1: /CLK8 -> /CLK8M
- JP1 pad 3: /CLK8_O -> /CLK8O
- R1 pad 2: Net-(J14-Pin_1) -> /CONFIG2
- R3 pad 1: Net-(J5-Pin_9) -> +5V
- R3 pad 2: GND -> /CONFIG1
- R4 pad 1: Net-(J6-Pin_9) -> +5V
- R4 pad 2: GND -> /CONFIG0
- U1 pad 1: /D4 -> /DI4
- U1 pad 10: /~{DTACK} -> /~{DTACK}I
- U1 pad 11: /~{BG_I} -> /~{BG}I
- U1 pad 12: /~{BGACK_I} -> /~{BGACK}I
- U1 pad 13: /~{BR_I} -> /~{BR}I
- U1 pad 17: /~{HALT_I} -> /~{HALT}I
- U1 pad 18: /~{RESET_I} -> /~{RESET}
- U1 pad 19: /~{VMA} -> /~{VMA}I
- U1 pad 2: /D3 -> /DI3
- U1 pad 20: /E -> unconnected-(U1-E-Pad20)
- U1 pad 21: /~{VPA} -> /~{VPA}I
- U1 pad 22: /~{BERR} -> /~{BERR}I
- U1 pad 26: /~{FC2} -> /~{FC2}I
- U1 pad 27: /~{FC1} -> /~{FC1}I
- U1 pad 28: /~{FC0} -> /~{FC0}I
- U1 pad 29: /A1 -> /AI1
- U1 pad 3: /D2 -> /DI2
- U1 pad 30: /A2 -> /AI2
- U1 pad 31: /A3 -> /AI3
- U1 pad 32: /A4 -> /AI4
- U1 pad 33: /A5 -> /AI5
- U1 pad 34: /A6 -> /AI6
- U1 pad 35: /A7 -> /AI7
- U1 pad 36: /A8 -> /AI8
- U1 pad 37: /A9 -> /AI9
- U1 pad 38: /A10 -> /AI10
- U1 pad 39: /A11 -> /AI11
- U1 pad 4: /D1 -> /DI1
- U1 pad 40: /A12 -> /AI12
- U1 pad 41: /A13 -> /AI13
- U1 pad 42: /A14 -> /AI14
- U1 pad 43: /A15 -> /AI15
- U1 pad 44: /A16 -> /AI16
- U1 pad 45: /A17 -> /AI17
- U1 pad 46: /A18 -> /AI18
- U1 pad 47: /A19 -> /AI19
- U1 pad 48: /A20 -> /AI20
- U1 pad 5: /D0 -> /DI0
- U1 pad 50: /A21 -> /AI21
- U1 pad 51: /A22 -> /AI22
- U1 pad 52: /A23 -> /AI23
- U1 pad 54: /D15 -> /DI15
- U1 pad 55: /D14 -> /DI14
- U1 pad 56: /D13 -> /DI13
- U1 pad 57: /D12 -> /DI12
- U1 pad 58: /D11 -> /DI11
- U1 pad 59: /D10 -> /DI10
- U1 pad 6: /~{AS} -> /~{AS}I
- U1 pad 60: /D9 -> /DI9
- U1 pad 61: /D8 -> /DI8
- U1 pad 62: /D7 -> /DI7
- U1 pad 63: /D6 -> /DI6
- U1 pad 64: /D5 -> /DI5
- U1 pad 7: /~{UDS} -> /~{UDS}I
- U1 pad 8: /~{LDS} -> /~{LDS}I
- U1 pad 9: /R~{W} -> /R~{W}I
- U3 pad 1: unconnected-(U3-I/O/GCK3-Pad1) -> /EM
- U3 pad 12: unconnected-(U3-I/O-Pad12) -> /~{VMA}M
- U3 pad 14: unconnected-(U3-I/O-Pad14) -> /CONFIG0
- U3 pad 16: unconnected-(U3-I/O-Pad16) -> /CONFIG1
- U3 pad 18: unconnected-(U3-I/O-Pad18) -> /CONFIG2
- U3 pad 2: unconnected-(U3-I/O-Pad2) -> /~{AS}I
- U3 pad 20: unconnected-(U3-I/O-Pad20) -> /~{HALT_MB}M
- U3 pad 23: unconnected-(U3-I/O-Pad23) -> /~{BR_MB}M
- U3 pad 27: unconnected-(U3-I/O-Pad27) -> /~{BG_MB}M
- U3 pad 28: unconnected-(U3-I/O-Pad28) -> /~{BGACK_MB}M
- U3 pad 29: /~{RESET_MB_CPLD} -> /~{RESET}
- U3 pad 3: unconnected-(U3-I/O-Pad3) -> /~{DTACK}I
- U3 pad 30: /~{HALT_MB_CPLD} -> /~{HALT}I
- U3 pad 31: /~{BR_MB_CPLD} -> /~{FC0}I
- U3 pad 32: /~{BGACK_MB_CPLD} -> /~{FC1}I
- U3 pad 33: /~{BG_MB_CPLD} -> /~{BR}I
- U3 pad 34: /~{BG_I_CPLD} -> /~{BG}I
- U3 pad 36: /~{BGACK_I_CPLD} -> /~{BGACK}I
- U3 pad 37: /~{BR_I_CPLD} -> unconnected-(U3-I/O-Pad37)
- U3 pad 38: /~{HALT_I_CPLD} -> /ISOLATION
- U3 pad 39: /~{RESET_I_CPLD} -> /~{VPA}I
- U3 pad 42: unconnected-(U3-I/O-Pad42) -> /CLK8O
- U3 pad 43: /CLK8_O -> /CLK8M
- U3 pad 44: /CLK8 -> /OSC
- U3 pad 6: unconnected-(U3-I/O-Pad6) -> /~{AS}M
- U3 pad 7: unconnected-(U3-I/O-Pad7) -> /~{DTACK}M
- U3 pad 8: unconnected-(U3-I/O-Pad8) -> /~{VPA}M
Routing:
- net +5V: track 489.3 -> 0.00 mm, vias 7 -> 0
- net /CLK8I: track 285.0 -> 0.00 mm, vias 1 -> 0
- net /~{IPL1}: track 101.6 -> 0.00 mm
- net /~{RESET_MB}: track 99.1 -> 0.00 mm, vias 1 -> 0
- net /~{HALT_MB}: track 98.2 -> 0.00 mm, vias 1 -> 0
- net /~{IPL2}: track 96.2 -> 0.00 mm
- net /~{RESET_I}: track 93.9 -> 0.00 mm, vias 2 -> 0
- net /~{HALT_I}: track 90.7 -> 0.00 mm, vias 2 -> 0
- net /~{BR_MB}: track 85.7 -> 0.00 mm, vias 1 -> 0
- net /~{BGACK_MB}: track 84.8 -> 0.00 mm, vias 1 -> 0
- net /~{BG_MB}: track 84.3 -> 0.00 mm, vias 1 -> 0
- net /~{BR_I}: track 76.3 -> 0.00 mm
- net /~{BGACK_I}: track 72.7 -> 0.00 mm
- net /CLK8: track 72.2 -> 0.00 mm, vias 1 -> 0
- net /~{BG_I}: track 69.1 -> 0.00 mm
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Other:
- board text removed: "RESET_I HALT_I BR_I BGK_I BG_I BG_MB BGK_MB BR_MB HALT_MB RESET_MB"
