File: kicad/megabusmaster.kicad_sch (KiCad schematic)
At the start: 46 parts, among them J1 Conn_02x32_Odd_Even, J10 Conn_01x08_Pin, J11 Conn_01x13_Pin, J12 Conn_01x13_Pin, J13 Conn_01x06_Pin, J14 Conn_01x04_Pin, J15 Conn_01x02_Pin, J2 Conn_01x06_Pin, J3 Conn_02x04_Odd_Even, J4 Conn_02x10_Odd_Even, J5 Conn_01x09_Pin, J6 Conn_01x09_Pin, J7 Conn_01x08_Pin, J8 Conn_01x08_Pin, J9 Conn_01x08_Pin, U1 MC68000P, U2 LM1117T-3.3, U3 XC9572XL-xxVQx44, U4 GAL16V8, U5 GAL16V8, U6 GAL20V8, U7 GAL20V8

Commit message: Work commenced on second revision
Parts:
- removed C6, C7, C8, C9: 100n, Capacitor_SMD:C_0805_2012Metric_Pad1.18x1.45mm_HandSolder, symbol Device:C
- removed J10, J7, J8, J9: Conn_01x08_Pin, Connector_PinHeader_2.54mm:PinHeader_1x08_P2.54mm_Vertical, symbol Connector:Conn_01x08_Pin
- removed J11, J12: Conn_01x13_Pin, Connector_PinHeader_2.54mm:PinHeader_1x13_P2.54mm_Vertical, symbol Connector:Conn_01x13_Pin
- removed J14: Conn_01x04_Pin, Connector_PinHeader_2.54mm:PinHeader_1x04_P2.54mm_Vertical, symbol Connector:Conn_01x04_Pin
- removed J4: Conn_02x10_Odd_Even, Connector_PinHeader_2.54mm:PinHeader_2x10_P2.54mm_Vertical, symbol Connector_Generic:Conn_02x10_Odd_Even
- removed J5, J6: Conn_01x09_Pin, Connector_PinHeader_2.54mm:PinHeader_1x09_P2.54mm_Vertical, symbol Connector:Conn_01x09_Pin
- removed R1, R3, R4, R5, R6: 10k, Resistor_SMD:R_0805_2012Metric_Pad1.20x1.40mm_HandSolder, symbol Device:R
- removed U4, U5: GAL16V8, Package_DIP:DIP-20_W7.62mm_Socket_LongPads, symbol Logic_Programmable:GAL16V8
- removed U6, U7: GAL20V8, Package_DIP:DIP-24_W7.62mm_Socket_LongPads, symbol megabusmaster:GAL20V8
- added IC1, IC2, IC3: SN74CB3T3245PW, SOP65P640X110-20N, symbol SN74CB3T3245PW:SN74CB3T3245PW
- R2: value 10k -> 1k
Connections:
- net CLK8_O is gone; now on net CLK8O: JP1.3 (B), U3.43 (I/O/GCK1)
- net CLK8O: now reaches U3.42 (I/O)
- net A1 renamed AI1
- net AI1: no longer J1.57 (Pin_57)
- net A10 renamed AI10
- net AI10: no longer J1.54 (Pin_54)
- net A11 renamed AI11
- net AI11: no longer J1.52 (Pin_52)
- net A12 renamed AI12
- net AI12: no longer J1.50 (Pin_50)
- net A13 renamed AI13
- net AI13: no longer J1.48 (Pin_48)
- net A14 renamed AI14
- net AI14: no longer J1.46 (Pin_46)
- net A15 renamed AI15
- net AI15: no longer J1.44 (Pin_44)
- net A16 renamed AI16
- net AI16: no longer J1.42 (Pin_42)
- net A17 renamed AI17
- net AI17: no longer J1.40 (Pin_40)
- net A18 renamed AI18
- net AI18: no longer J1.38 (Pin_38)
- net A19 renamed AI19
- net AI19: no longer J1.36 (Pin_36)
- net A2 renamed AI2
- net AI2: no longer J1.59 (Pin_59)
- net A20 renamed AI20
- net AI20: no longer J1.34 (Pin_34)
- net A21 renamed AI21
- net AI21: no longer J1.30 (Pin_30)
- net A22 renamed AI22
- net AI22: no longer J1.28 (Pin_28)
- net A23 renamed AI23
- net AI23: no longer J1.26 (Pin_26)
- net A3 renamed AI3
- net AI3: no longer J1.61 (Pin_61)
- net A4 renamed AI4
- net AI4: no longer J1.63 (Pin_63)
- net A5 renamed AI5
- net AI5: no longer J1.64 (Pin_64)
- net A6 renamed AI6
- net AI6: no longer J1.62 (Pin_62)
- net A7 renamed AI7
- net AI7: no longer J1.60 (Pin_60)
- net A8 renamed AI8
- net AI8: no longer J1.58 (Pin_58)
- net A9 renamed AI9
- net AI9: no longer J1.56 (Pin_56)
- net CLK8 renamed CLK8M
- net CLK8_I renamed CLK8I
- net D0 renamed DI0
- net DI0: no longer J1.9 (Pin_9)
- net D1 renamed DI1
- net DI1: no longer J1.7 (Pin_7)
- net D10 renamed DI10
- net DI10: no longer J1.12 (Pin_12)
- net D11 renamed DI11
- net DI11: no longer J1.14 (Pin_14)
- net D12 renamed DI12
- net DI12: no longer J1.16 (Pin_16)
- net D13 renamed DI13
- net DI13: no longer J1.18 (Pin_18)
- net D14 renamed DI14
- net DI14: no longer J1.20 (Pin_20)
- net D15 renamed DI15
- net DI15: no longer J1.22 (Pin_22)
- net D2 renamed DI2
- net DI2: no longer J1.5 (Pin_5)
- net D3 renamed DI3
- net DI3: no longer J1.3 (Pin_3)
- net D4 renamed DI4
- net DI4: no longer J1.1 (Pin_1)
- net D5 renamed DI5
- net DI5: no longer J1.2 (Pin_2)
- net D6 renamed DI6
- net DI6: no longer J1.4 (Pin_4)
- net D7 renamed DI7
- net DI7: no longer J1.6 (Pin_6)
- net D8 renamed DI8
- net DI8: no longer J1.8 (Pin_8)
- net D9 renamed DI9
- net DI9: no longer J1.10 (Pin_10)
- net E: no longer names the net of U1.20 (E)
- net E: no longer J1.39 (Pin_39)
- net R~{W} renamed R~{W}I
- net R~{W}I: no longer J1.17 (Pin_17)
- net ~{AS} renamed ~{AS}I
- net ~{AS}I: no longer J1.11 (Pin_11)
- net ~{BERR} renamed ~{BERR}I
- net ~{BERR}I: no longer J1.43 (Pin_43)
- net ~{BGACK_I_CPLD}: no longer names the net of U3.36 (I/O/GTS1)
- net ~{BGACK_I} renamed ~{BGACK}I
- net ~{BGACK_MB_CPLD}: no longer names the net of U3.32 (I/O)
- net ~{BGACK_MB} renamed ~{BGACK_MB}M
- net ~{BG_I_CPLD}: no longer names the net of U3.34 (I/O/GTS2)
- net ~{BG_I} renamed ~{BG}I
- net ~{BG_MB_CPLD}: no longer names the net of U3.33 (I/O/GSR)
- net ~{BG_MB} renamed ~{BG_MB}M
- net ~{BR_I_CPLD}: no longer names the net of U3.37 (I/O)
- net ~{BR_I} renamed ~{BR}I
- net ~{BR_MB_CPLD}: no longer names the net of U3.31 (I/O)
- net ~{BR_MB} renamed ~{BR_MB}M
- net ~{DTACK} renamed ~{DTACK}I
- net ~{DTACK}I: no longer J1.19 (Pin_19)
- net ~{FC0} renamed ~{FC0}I
- net ~{FC0}I: no longer J1.55 (Pin_55)
- net ~{FC1} renamed ~{FC1}I
- net ~{FC1}I: no longer J1.53 (Pin_53)
- net ~{FC2} renamed ~{FC2}I
- net ~{FC2}I: no longer J1.51 (Pin_51)
- net ~{HALT_I_CPLD}: no longer names the net of U3.38 (I/O)
- net ~{HALT_I} renamed ~{HALT}I
- net ~{HALT_MB_CPLD}: no longer names the net of U3.30 (I/O)
- net ~{HALT_MB} renamed ~{HALT_MB}M
- net ~{LDS} renamed ~{LDS}I
- net ~{LDS}I: no longer J1.15 (Pin_15)
- net ~{RESET_I_CPLD}: no longer names the net of U3.39 (I/O)
- net ~{RESET_I} renamed ~{RESET}
- net ~{RESET_MB_CPLD}: no longer names the net of U3.29 (I/O)
- net ~{RESET_MB} renamed ~{RESET_MB}M
- net ~{UDS} renamed ~{UDS}I
- net ~{UDS}I: no longer J1.13 (Pin_13)
- net ~{VMA} renamed ~{VMA}I
- net ~{VMA}I: no longer J1.37 (Pin_37)
- net ~{VPA} renamed ~{VPA}I
- net ~{VPA}I: no longer J1.41 (Pin_41)
- new net AM1: J1.57 (Pin_57)
- new net AM10: J1.54 (Pin_54)
- new net AM11: J1.52 (Pin_52)
- new net AM12: J1.50 (Pin_50)
- new net AM13: J1.48 (Pin_48)
- new net AM14: J1.46 (Pin_46)
- new net AM15: J1.44 (Pin_44)
- new net AM16: J1.42 (Pin_42)
- new net AM17: J1.40 (Pin_40)
- new net AM18: J1.38 (Pin_38)
- new net AM19: J1.36 (Pin_36)
- new net AM2: J1.59 (Pin_59)
- new net AM20: J1.34 (Pin_34)
- new net AM21: J1.30 (Pin_30)
- new net AM22: J1.28 (Pin_28)
- new net AM23: J1.26 (Pin_26)
- new net AM3: J1.61 (Pin_61)
- new net AM4: J1.63 (Pin_63)
- new net AM5: J1.64 (Pin_64)
- new net AM6: J1.62 (Pin_62)
- new net AM7: J1.60 (Pin_60)
- new net AM8: J1.58 (Pin_58)
- new net AM9: J1.56 (Pin_56)
- new net DM0: J1.9 (Pin_9)
- new net DM1: J1.7 (Pin_7)
- new net DM10: J1.12 (Pin_12)
- new net DM11: J1.14 (Pin_14)
- new net DM12: J1.16 (Pin_16)
- new net DM13: J1.18 (Pin_18)
- new net DM14: J1.20 (Pin_20)
- new net DM15: J1.22 (Pin_22)
- new net DM2: J1.5 (Pin_5)
- new net DM3: J1.3 (Pin_3)
- new net DM4: J1.1 (Pin_1)
- new net DM5: J1.2 (Pin_2)
- new net DM6: J1.4 (Pin_4)
- new net DM7: J1.6 (Pin_6)
- new net DM8: J1.8 (Pin_8)
- new net DM9: J1.10 (Pin_10)
- new net EM: J1.39 (Pin_39)
- new net R~{W}M: J1.17 (Pin_17)
- new net ~{AS}M: J1.11 (Pin_11)
- new net ~{BERR}M: J1.43 (Pin_43)
- new net ~{DTACK}M: J1.19 (Pin_19)
- new net ~{FC0}M: J1.55 (Pin_55)
- new net ~{FC1}M: J1.53 (Pin_53)
- new net ~{FC2}M: J1.51 (Pin_51)
- new net ~{LDS}M: J1.15 (Pin_15)
- new net ~{UDS}M: J1.13 (Pin_13)
- new net ~{VMA}M: J1.37 (Pin_37)
- new net ~{VPA}M: J1.41 (Pin_41)
- no-connect marks 22 -> 23
Other:
- moved on the sheet: C1, C10, C11, C12, C2, C3, C4, C5, H1, H2, H3, H4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

Commit message: Initial attempt at second revision schematic.
Parts:
- added C6: 100n, Oscillator:Oscillator_DIP-14, symbol Device:C
- added IC4, IC5, IC6: SN74CB3T3245PW, SOP65P640X110-20N, symbol SN74CB3T3245PW:SN74CB3T3245PW
- added J4: Conn_02x07_Counter_Clockwise, Package_QFP:TQFP-44_10x10mm_P0.8mm, symbol Connector_Generic:Conn_02x07_Counter_Clockwise
- added J5: Conn_02x03_Odd_Even, symbol Connector_Generic:Conn_02x03_Odd_Even
- added R1, R3, R4: 10k, symbol Device:R
- added R10, R8, R9: 10k, Resistor_SMD:R_0805_2012Metric_Pad1.20x1.40mm_HandSolder, symbol Device:R
Connections:
- net +5V: now also C6.1, J4.14 (Pin_14), R1.1, R10.1, R3.1, R4.1, R8.1, R9.1
- net AI1: now also IC3.11 (B8)
- net AI10: now also IC2.12 (B7)
- net AI11: now also IC2.13 (B6)
- net AI12: now also IC2.14 (B5)
- net AI13: now also IC2.15 (B4)
- net AI14: now also IC2.16 (B3)
- net AI15: now also IC2.17 (B2)
- net AI16: now also IC2.18 (B1)
- net AI17: now also IC1.11 (B8)
- net AI18: now also IC1.12 (B7)
- net AI19: now also IC1.13 (B6)
- net AI2: now also IC3.12 (B7)
- net AI20: now also IC1.14 (B5)
- net AI21: now also IC1.15 (B4)
- net AI22: now also IC1.16 (B3)
- net AI23: now also IC1.17 (B2)
- net AI3: now also IC3.13 (B6)
- net AI4: now also IC3.14 (B5)
- net AI5: now also IC3.15 (B4)
- net AI6: now also IC3.16 (B3)
- net AI7: now also IC3.17 (B2)
- net AI8: now also IC3.18 (B1)
- net AI9: now also IC2.11 (B8)
- net AM1: now also IC3.9 (A8)
- net AM10: now also IC2.8 (A7)
- net AM11: now also IC2.7 (A6)
- net AM12: now also IC2.6 (A5)
- net AM13: now also IC2.5 (A4)
- net AM14: now also IC2.4 (A3)
- net AM15: now also IC2.3 (A2)
- net AM16: now also IC2.2 (A1)
- net AM17: now also IC1.9 (A8)
- net AM18: now also IC1.8 (A7)
- net AM19: now also IC1.7 (A6)
- net AM2: now also IC3.8 (A7)
- net AM20: now also IC1.6 (A5)
- net AM21: now also IC1.5 (A4)
- net AM22: now also IC1.4 (A3)
- net AM23: now also IC1.3 (A2)
- net AM3: now also IC3.7 (A6)
- net AM4: now also IC3.6 (A5)
- net AM5: now also IC3.5 (A4)
- net AM6: now also IC3.4 (A3)
- net AM7: now also IC3.3 (A2)
- net AM8: now also IC3.2 (A1)
- net AM9: now also IC2.9 (A8)
- net CLK8M: now also U3.43 (I/O/GCK1); no longer U3.44 (I/O/GCK2)
- net CLK8O: no longer U3.43 (I/O/GCK1)
- net DI0: now also IC4.18 (B1)
- net DI1: now also IC4.17 (B2)
- net DI10: now also IC5.16 (B3)
- net DI11: now also IC5.15 (B4)
- net DI12: now also IC5.14 (B5)
- net DI13: now also IC5.13 (B6)
- net DI14: now also IC5.12 (B7)
- net DI15: now also IC5.11 (B8)
- net DI2: now also IC4.16 (B3)
- net DI3: now also IC4.15 (B4)
- net DI4: now also IC4.14 (B5)
- net DI5: now also IC4.13 (B6)
- net DI6: now also IC4.12 (B7)
- net DI7: now also IC4.11 (B8)
- net DI8: now also IC5.18 (B1)
- net DI9: now also IC5.17 (B2)
- net DM0: now also IC4.2 (A1)
- net DM1: now also IC4.3 (A2)
- net DM10: now also IC5.4 (A3)
- net DM11: now also IC5.5 (A4)
- net DM12: now also IC5.6 (A5)
- net DM13: now also IC5.7 (A6)
- net DM14: now also IC5.8 (A7)
- net DM15: now also IC5.9 (A8)
- net DM2: now also IC4.4 (A3)
- net DM3: now also IC4.5 (A4)
- net DM4: now also IC4.6 (A5)
- net DM5: now also IC4.7 (A6)
- net DM6: now also IC4.8 (A7)
- net DM7: now also IC4.9 (A8)
- net DM8: now also IC5.2 (A1)
- net DM9: now also IC5.3 (A2)
- net EM: now also U3.1 (I/O/GCK3)
- net GND: now also C6.2, J4.4 (Pin_4), J4.7 (Pin_7), J5.2 (Pin_2), J5.4 (Pin_4), J5.6 (Pin_6)
- net R~{W}I: now also IC1.18 (B1)
- net R~{W}M: now also IC1.2 (A1)
- net ~{AS}I: now also U3.2 (I/O), IC6.18 (B1)
- net ~{AS}M: now also U3.6 (I/O), IC6.2 (A1)
- net ~{BERR}I: now also IC6.11 (B8), R8.2
- net ~{BERR}M: now also IC6.9 (A8)
- net ~{BGACK_MB}M: now also U3.28 (I/O)
- net ~{BGACK}I: now also U3.36 (I/O/GTS1)
- net ~{BG_MB}M: now also U3.27 (I/O)
- net ~{BG}I: now also U3.34 (I/O/GTS2)
- net ~{BR_MB}M: now also U3.23 (I/O)
- net ~{BR}I: now also U3.33 (I/O/GSR)
- net ~{DTACK}I: now also U3.3 (I/O), IC6.15 (B4), R9.2
- net ~{DTACK}M: now also U3.7 (I/O), IC6.5 (A4)
- net ~{FC0}I: now also U3.31 (I/O), IC6.14 (B5)
- net ~{FC0}M: now also IC6.6 (A5)
- net ~{FC1}I: now also U3.32 (I/O), IC6.13 (B6)
- net ~{FC1}M: now also IC6.7 (A6)
- net ~{FC2}I: now also IC6.12 (B7)
- net ~{FC2}M: now also IC6.8 (A7)
- net ~{HALT_MB}M: now also U3.20 (I/O)
- net ~{HALT}I: now also U3.30 (I/O), R10.2
- net ~{LDS}I: now also IC6.16 (B3)
- net ~{LDS}M: now also IC6.4 (A3)
- net ~{RESET}: now also U3.29 (I/O)
- net ~{UDS}I: now also IC6.17 (B2)
- net ~{UDS}M: now also IC6.3 (A2)
- net ~{VPA}I: now also U3.39 (I/O)
- net ~{VPA}M: now also U3.8 (I/O)
- net CONFIG0: now reaches U3.14 (I/O)
- net CONFIG0: now also J5.1 (Pin_1), R4.2
- net CONFIG1: now reaches U3.16 (I/O)
- net CONFIG1: now also J5.3 (Pin_3), R3.2
- net CONFIG2: now reaches U3.18 (I/O)
- net CONFIG2: now also J5.5 (Pin_5), R1.2
- new net OSC: J4.11 (Pin_11), J4.8 (Pin_8), U3.44 (I/O/GCK2)
- no-connect marks 23 -> 15
Other:
- moved on the sheet: C10, C11, C12, C3, C4, C5, H1, H2, H3, H4, IC1, IC2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

Commit message: Started board layout of rev2
Parts:
- added C13, C14, C15, C7, C8, C9: 100n, Capacitor_SMD:C_0805_2012Metric_Pad1.18x1.45mm_HandSolder, symbol Device:C
- C6: footprint Oscillator:Oscillator_DIP-14 -> Capacitor_SMD:C_0805_2012Metric_Pad1.18x1.45mm_HandSolder
- IC1, IC2, IC3, IC4, IC5, IC6: footprint SOP65P640X110-20N -> Package_SO:TSSOP-20_4.4x6.5mm_P0.65mm
- J4: footprint Package_QFP:TQFP-44_10x10mm_P0.8mm -> Package_DIP:DIP-14_W7.62mm_Socket
- J5: footprint (none) -> Connector_PinHeader_2.54mm:PinHeader_2x03_P2.54mm_Vertical
- R1, R3, R4: footprint (none) -> Resistor_SMD:R_0805_2012Metric_Pad1.20x1.40mm_HandSolder
Connections:
- net ~{RESET_MB}M is gone; now on net ~{RESET}: J1.35 (Pin_35)
- net +5V: now also IC1.20 (VCC), IC2.20 (VCC), IC3.20 (VCC), IC4.20 (VCC), IC5.20 (VCC), IC6.20 (VCC), C13.1, C14.1, C15.1, C7.1, C8.1, C9.1
- net AI14: now also IC1.11 (B8); no longer IC2.16 (B3)
- net AI15: now also IC1.12 (B7); no longer IC2.17 (B2)
- net AI16: now also IC1.14 (B5); no longer IC2.18 (B1)
- net AI17: now also IC1.15 (B4); no longer IC1.11 (B8)
- net AI18: now also IC1.16 (B3); no longer IC1.12 (B7)
- net AI19: now also IC1.17 (B2); no longer IC1.13 (B6)
- net AI20: now also IC1.18 (B1); no longer IC1.14 (B5)
- net AI21: now also IC6.11 (B8); no longer IC1.15 (B4)
- net AI22: now also IC6.12 (B7); no longer IC1.16 (B3)
- net AI23: now also IC6.13 (B6); no longer IC1.17 (B2)
- net AM14: now also IC1.9 (A8); no longer IC2.4 (A3)
- net AM15: now also IC1.8 (A7); no longer IC2.3 (A2)
- net AM16: now also IC1.6 (A5); no longer IC2.2 (A1)
- net AM17: now also IC1.5 (A4); no longer IC1.9 (A8)
- net AM18: now also IC1.4 (A3); no longer IC1.8 (A7)
- net AM19: now also IC1.3 (A2); no longer IC1.7 (A6)
- net AM20: now also IC1.2 (A1); no longer IC1.6 (A5)
- net AM21: now also IC6.9 (A8); no longer IC1.5 (A4)
- net AM22: now also IC6.8 (A7); no longer IC1.4 (A3)
- net AM23: now also IC6.7 (A6); no longer IC1.3 (A2)
- net DI0: now also IC5.17 (B2); no longer IC4.18 (B1)
- net DI1: now also IC4.12 (B7); no longer IC4.17 (B2)
- net DI10: now also IC5.15 (B4); no longer IC5.16 (B3)
- net DI11: now also IC5.13 (B6); no longer IC5.15 (B4)
- net DI12: now also IC5.11 (B8); no longer IC5.14 (B5)
- net DI13: now also IC6.18 (B1); no longer IC5.13 (B6)
- net DI14: now also IC6.16 (B3); no longer IC5.12 (B7)
- net DI15: now also IC6.14 (B5); no longer IC5.11 (B8)
- net DI2: now also IC4.14 (B5); no longer IC4.16 (B3)
- net DI3: now also IC4.16 (B3); no longer IC4.15 (B4)
- net DI4: now also IC4.17 (B2); no longer IC4.14 (B5)
- net DI5: now also IC4.18 (B1); no longer IC4.13 (B6)
- net DI6: now also IC4.15 (B4); no longer IC4.12 (B7)
- net DI7: now also IC4.13 (B6); no longer IC4.11 (B8)
- net DI8: now also IC4.11 (B8); no longer IC5.18 (B1)
- net DI9: now also IC5.18 (B1); no longer IC5.17 (B2)
- net DM0: now also IC5.3 (A2); no longer IC4.2 (A1)
- net DM1: now also IC4.8 (A7); no longer IC4.3 (A2)
- net DM10: now also IC5.5 (A4); no longer IC5.4 (A3)
- net DM11: now also IC5.7 (A6); no longer IC5.5 (A4)
- net DM12: now also IC5.9 (A8); no longer IC5.6 (A5)
- net DM13: now also IC6.2 (A1); no longer IC5.7 (A6)
- net DM14: now also IC6.4 (A3); no longer IC5.8 (A7)
- net DM15: now also IC6.6 (A5); no longer IC5.9 (A8)
- net DM2: now also IC4.6 (A5); no longer IC4.4 (A3)
- net DM3: now also IC4.4 (A3); no longer IC4.5 (A4)
- net DM4: now also IC4.3 (A2); no longer IC4.6 (A5)
- net DM5: now also IC4.2 (A1); no longer IC4.7 (A6)
- net DM6: now also IC4.5 (A4); no longer IC4.8 (A7)
- net DM7: now also IC4.7 (A6); no longer IC4.9 (A8)
- net DM8: now also IC4.9 (A8); no longer IC5.2 (A1)
- net DM9: now also IC5.2 (A1); no longer IC5.3 (A2)
- net GND: now also IC1.10 (GND), IC2.10 (GND), IC3.10 (GND), IC4.10 (GND), IC5.10 (GND), IC6.10 (GND), C13.2, C14.2, C15.2, C7.2, C8.2, C9.2
- net R~{W}I: now also IC6.17 (B2); no longer IC1.18 (B1)
- net R~{W}M: now also IC6.3 (A2); no longer IC1.2 (A1)
- net ~{AS}I: now also IC5.16 (B3); no longer IC6.18 (B1)
- net ~{AS}M: now also IC5.4 (A3); no longer IC6.2 (A1)
- net ~{BERR}I: now also IC1.13 (B6); no longer IC6.11 (B8)
- net ~{BERR}M: now also IC1.7 (A6); no longer IC6.9 (A8)
- net ~{FC0}I: no longer IC6.14 (B5)
- net ~{FC0}M: no longer IC6.6 (A5)
- net ~{FC1}I: no longer IC6.13 (B6)
- net ~{FC1}M: no longer IC6.7 (A6)
- net ~{FC2}I: no longer IC6.12 (B7)
- net ~{FC2}M: no longer IC6.8 (A7)
- net ~{LDS}I: now also IC5.12 (B7); no longer IC6.16 (B3)
- net ~{LDS}M: now also IC5.8 (A7); no longer IC6.4 (A3)
- net ~{UDS}I: now also IC5.14 (B5); no longer IC6.17 (B2)
- net ~{UDS}M: now also IC5.6 (A5); no longer IC6.3 (A2)
- net ~{VMA}M: now also U3.12 (I/O)
- net ISOLATION: now reaches IC2.19 (~{OE})
- net ISOLATION: now also IC1.19 (~{OE}), IC3.19 (~{OE}), IC4.19 (~{OE}), IC5.19 (~{OE}), IC6.19 (~{OE}), U3.38 (I/O)
- no-connect marks 15 -> 23
